File: Key Matrix.sch (KiCad schematic (older format))
At the start: 174 parts

Commit message: Update matrix and MCU
Updated matrix. Added decoupling capacitors. Added Encoder.
Parts:
- MX?: renamed from TAB; value MX-NoLED -> TAB
- MX?: renamed from Q; value MX-NoLED -> Q
- MX?: renamed from W; value MX-NoLED -> W
- MX?: renamed from E; value MX-NoLED -> E
- MX?: renamed from R; value MX-NoLED -> R
- MX?: renamed from T; value MX-NoLED -> T
- MX?: renamed from Y; value MX-NoLED -> Y
- MX?: renamed from U; value MX-NoLED -> U
- MX?: renamed from I; value MX-NoLED -> I
- MX?: renamed from O; value MX-NoLED -> O
- MX?: renamed from P; value MX-NoLED -> P
- MX?: renamed from [; value MX-NoLED -> [
- MX?: renamed from ]; value MX-NoLED -> ]
- MX?: renamed from \; value MX-NoLED -> \\
- MX?: renamed from DEL; value MX-NoLED -> DEL
- MX?: renamed from CAPLK; value MX-NoLED -> CAP_LK
- MX?: renamed from A; value MX-NoLED -> A
- MX?: renamed from S; value MX-NoLED -> S
- MX?: renamed from D; value MX-NoLED -> D
- MX?: renamed from F; value MX-NoLED -> F
- MX?: renamed from G; value MX-NoLED -> G
- MX?: renamed from H; value MX-NoLED -> H
- MX?: renamed from J; value MX-NoLED -> J
- MX?: renamed from K; value MX-NoLED -> K
- MX?: renamed from L; value MX-NoLED -> L
- MX?: renamed from ;; value MX-NoLED -> ;
- MX?: renamed from '; value MX-NoLED -> '
- MX?: renamed from ENTER; value MX-NoLED -> ENTER
- MX?: renamed from L_SHIFT; value MX-NoLED -> L_SHIFT
- MX?: renamed from Z; value MX-NoLED -> Z
- MX?: renamed from X; value MX-NoLED -> X
- MX?: renamed from C; value MX-NoLED -> C
- MX?: renamed from V; value MX-NoLED -> V
- MX?: renamed from B; value MX-NoLED -> B
- MX?: renamed from N; value MX-NoLED -> N
- MX?: renamed from M; value MX-NoLED -> M
- MX?: renamed from ,; value MX-NoLED -> ,
- MX?: renamed from .; value MX-NoLED -> .
- MX?: renamed from /; value MX-NoLED -> /
- MX?: renamed from R_SHIFT; value MX-NoLED -> R_SHIFT
- MX?: renamed from UP; value MX-NoLED -> UP
- MX?: renamed from L_CTRL; value MX-NoLED -> L_CTRL
- MX?: renamed from L_OS; value MX-NoLED -> L_OS
- MX?: renamed from L_ALT; value MX-NoLED -> L_ALT
- MX?: renamed from SPACE; value MX-NoLED -> SPACE
- MX?: renamed from R_ALT; value MX-NoLED -> R_ALT
- MX?: renamed from R_OS; value MX-NoLED -> R_OS
- MX?: renamed from R_FN; value MX-NoLED -> R_FN
- MX?: renamed from R_CTRL; value MX-NoLED -> R_CTRL
- MX?: renamed from LEFT; value MX-NoLED -> LEFT
- MX?: renamed from DOWN; value MX-NoLED -> DOWN
- MX?: renamed from RIGHT; value MX-NoLED -> RIGHT

Commit message: Begin annotation
Annotated schematic and began associating symbols with footprints.
Parts:
- gave numbers to parts that had none: 174

Commit message: Assign Footprints
Continued assigning footprints
Parts:
- D10, D11, D12, D13, D14, D15, D16, D17, D18, D19, D20, D21, D22, D23, D24, D25, D26, D27, D28, D29, D30, D31, D32, D33, D34, D35, D36, D37, D38, D39, D4, D40, D41, D42, D43, D44, D45, D46, D47, D48, D49, D5, D50, D51, D52, D53, D54, D55, D56, D57, D58, D59, D6, D60, D61, D62, D63, D64, D65, D66, D67, D68, D69, D7, D70, D71, D72, D73, D74, D75, D76, D77, D78, D79, D8, D80, D81, D82, D83, D84, D85, D86, D87, D88, D89, D9, D90: footprint (none) -> Diode_SMD:D_0805_2012Metric

Commit message: Associate FP
added debounce to encoder. finalized footrpint association.
Parts:
- D10, D11, D12, D13, D14, D15, D16, D17, D18, D19, D20, D21, D22, D23, D24, D25, D26, D27, D28, D29, D30, D31, D32, D33, D34, D35, D36, D37, D38, D39, D4, D40, D41, D42, D43, D44, D45, D46, D47, D48, D49, D5, D50, D51, D52, D53, D54, D55, D56, D57, D58, D59, D6, D60, D61, D62, D63, D64, D65, D66, D67, D68, D69, D7, D70, D71, D72, D73, D74, D75, D76, D77, D78, D79, D8, D80, D81, D82, D83, D84, D85, D86, D87, D88, D89, D9, D90: footprint Diode_SMD:D_0805_2012Metric -> Diode_SMD:D_SOD-123
- MX1, MX10, MX11, MX12, MX13, MX14, MX15, MX16, MX17, MX18, MX19, MX2, MX20, MX21, MX22, MX23, MX24, MX25, MX26, MX27, MX28, MX29, MX3, MX31, MX32, MX33, MX35, MX36, MX37, MX38, MX39, MX4, MX40, MX41, MX42, MX43, MX44, MX45, MX46, MX48, MX49, MX5, MX50, MX52, MX53, MX54, MX55, MX56, MX57, MX58, MX59, MX6, MX60, MX61, MX62, MX65, MX66, MX67, MX68, MX69, MX7, MX70, MX71, MX72, MX73, MX74, MX76, MX8, MX85, MX86, MX87, MX9: footprint (none) -> 1_MX_Only:MXOnly-1U-Hotswap
- MX30: footprint (none) -> 1_MX_Only:MXOnly-2U-Hotswap
- MX34, MX47: footprint (none) -> 1_MX_Only:MXOnly-1.5U-Hotswap
- MX51: footprint (none) -> 1_MX_Only:MXOnly-1.75U-Hotswap
- MX63, MX64: footprint (none) -> 1_MX_Only:MXOnly-2.25U-Hotswap
- MX75: footprint (none) -> 1_MX_Only:MXOnly-2.75U-Hotswap
- MX77, MX78, MX79, MX81, MX82, MX83, MX84: footprint (none) -> 1_MX_Only:MXOnly-1.25U-Hotswap
- MX80: footprint (none) -> 1_MX_Only:MXOnly-6.25U-Hotswap

Commit message: usb layout
Connections:
- net COL5: now also MX80.1 (COL)
- net COL6: no longer MX80.1 (COL)
Other:
- moved on the sheet: D83, MX80
Changed lines of the file:
@@
 	10250 6100 10100 6100
 Wire Wire Line
-	5150 6100 5000 6100
+	4600 6100 4450 6100
 $Comp
 L Device:D D83
 U 1 1 5F521CD3
-P 5000 6250
-F 0 "D83" V 5046 6170 50  0000 R CNN
-F 1 "D" V 4955 6170 50  0000 R CNN
-F 2 "Diode_SMD:D_SOD-123" H 5000 6250 50  0001 C CNN
-F 3 "~" H 5000 6250 50  0001 C CNN
-	1    5000 6250
+P 4450 6250
+F 0 "D83" V 4496 6170 50  0000 R CNN
+F 1 "D" V 4405 6170 50  0000 R CNN
+F 2 "Diode_SMD:D_SOD-123" H 4450 6250 50  0001 C CNN
+F 3 "~" H 4450 6250 50  0001 C CNN
+	1    4450 6250
 	0    -1   -1   0
 $EndComp
@@
 L 1_MX_Alps_Hybrid:MX-NoLED MX80
 U 1 1 5F521CC9
-P 5200 5950
-F 0 "MX80" H 5233 6173 60  0000 C CNN
-F 1 "SPACE" H 5233 6099 20  0000 C CNN
-F 2 "1_MX_Only:MXOnly-6.25U-Hotswap" H 4575 5925 60  0001 C CNN
-F 3 "" H 4575 5925 60  0001 C CNN
-	1    5200 5950
+P 4650 5950
+F 0 "MX80" H 4683 6173 60  0000 C CNN
+F 1 "SPACE" H 4683 6099 20  0000 C CNN
+F 2 "1_MX_Only:MXOnly-6.25U-Hotswap" H 4025 5925 60  0001 C CNN
+F 3 "" H 4025 5925 60  0001 C CNN
+	1    4650 5950
 	1    0    0    -1
 $EndComp
@@
 Wire Wire Line
 	5350 2600 5350 3450
-Connection ~ 5350 5100
-Wire Wire Line
-	5350 5100 5350 5900
 Connection ~ 5350 4300
 Wire Wire Line
@@
 Wire Wire Line
 	2950 6400 2400 6400
-Connection ~ 5000 6400
-Wire Wire Line
-	5000 6400 2950 6400
 Connection ~ 7050 6400
-Wire Wire Line
-	7050 6400 5000 6400
 Connection ~ 7550 6400
 Wire Wire Line
@@
 	1    0    0    -1
 $EndComp
+Connection ~ 4450 6400
+Wire Wire Line
+	4450 6400 2950 6400
+Wire Wire Line
+	4450 6400 7050 6400
+Wire Wire Line
+	4800 5100 4800 5900
+Connection ~ 4800 5100
 $EndSCHEMATC

Commit message: Changed from hotswap to normal switch
Parts:
- MX1, MX10, MX11, MX12, MX13, MX14, MX15, MX16, MX17, MX18, MX19, MX2, MX20, MX21, MX22, MX23, MX24, MX25, MX26, MX27, MX28, MX29, MX3, MX31, MX32, MX33, MX35, MX36, MX37, MX38, MX39, MX4, MX40, MX41, MX42, MX43, MX44, MX45, MX46, MX48, MX49, MX5, MX50, MX52, MX53, MX54, MX55, MX56, MX57, MX58, MX59, MX6, MX60, MX61, MX62, MX65, MX66, MX67, MX68, MX69, MX7, MX70, MX71, MX72, MX73, MX74, MX76, MX8, MX85, MX86, MX87, MX9: footprint 1_MX_Only:MXOnly-1U-Hotswap -> 1_MX_Only:MXOnly-1U-NoLED
- MX30: footprint 1_MX_Only:MXOnly-2U-Hotswap -> 1_MX_Only:MXOnly-2U-NoLED
- MX34, MX47: footprint 1_MX_Only:MXOnly-1.5U-Hotswap -> 1_MX_Only:MXOnly-1.5U-NoLED
- MX51: footprint 1_MX_Only:MXOnly-1.75U-Hotswap -> 1_MX_Only:MXOnly-1.75U-NoLED
- MX63, MX64: footprint 1_MX_Only:MXOnly-2.25U-Hotswap -> 1_MX_Only:MXOnly-2.25U-NoLED
- MX75: footprint 1_MX_Only:MXOnly-2.75U-Hotswap -> 1_MX_Only:MXOnly-2.75U-NoLED
- MX77, MX78, MX79, MX82, MX83, MX84: footprint 1_MX_Only:MXOnly-1.25U-Hotswap -> 1_MX_Only:MXOnly-1.25U-NoLED
- MX80: footprint 1_MX_Only:MXOnly-6.25U-Hotswap -> 1_MX_Only:MXOnly-6.25U-NoLED
- MX81: footprint 1_MX_Only:MXOnly-1.25U-Hotswap -> 1_MX_Only:MXOnly-1.75U-NoLED

Commit message: Rotated switchs to south facing
Parts:
- MX81: footprint 1_MX_Only:MXOnly-1.75U-NoLED -> 1_MX_Only:MXOnly-1.25U-NoLED
Changed lines of the file:
@@
 F 0 "MX81" H 7283 6173 60  0000 C CNN
 F 1 "R_ALT" H 7283 6099 20  0000 C CNN
-F 2 "1_MX_Only:MXOnly-1.75U-NoLED" H 6625 5925 60  0001 C CNN
+F 2 "1_MX_Only:MXOnly-1.25U-NoLED" H 6625 5925 60  0001 C CNN
 F 3 "" H 6625 5925 60  0001 C CNN
 	1    7250 5950
