File: USB hub.sch (KiCad schematic (older format))
At the start: 33 parts, among them IC1 24SN, IC2 FE1.1S, J3 USB_A_SMT_FEMALE, J4 USB_A_SMT_FEMALE, P1 Lily58-cache_CONN_01X04, X1 12MHz

Commit message: refine sub hub
Connections:
- net D1-: now reaches D1.2 (IO1), IC2.10 (DM1), R14.1
- net D1+: now reaches D1.3 (IO2), IC2.11 (DP1), R15.1
- net D2-: now reaches D2.2 (IO1), IC2.8 (DM2), R20.1
- net D2+: now reaches D2.3 (IO2), IC2.9 (DP2), R21.1
Changed lines of the file:
@@
 NoConn ~ 6350 4850
 NoConn ~ 6350 4950
+Text Label 9900 4750 0    50   ~ 0
+D1-
+Text Label 9950 4850 0    50   ~ 0
+D1+
+Text Label 9950 6550 0    50   ~ 0
+D2-
+Text Label 9950 6650 0    50   ~ 0
+D2+
 $EndSCHEMATC
