File: Apex rev1.kicad_pcb (KiCad board)
At the start: 2 copper layers, 366.4 x 146.1 mm, 230 parts, among them IC1 24SN, IC2 FE1.1S, J1 OLED, J2 AVR-ISP-6, J3 USB_A_SMT_FEMALE, J4 USB_A_SMT_FEMALE, P1 Lily58-cache_CONN_01X04, SW1 SW_PUSH, SW2 Rotary_Encoder_Switch, U1 AT90USB1286-MU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

Commit message: silkscreen
Parts:
- added ?: , components:diode-silk, B.Cu at (59.9, 181.2)
- added ?: , components:diode-silk, B.Cu at (354.7, 188.1)
- added ?: , components:diode-silk, B.Cu at (373.5, 187.2)
- added ?: , components:diode-silk, B.Cu at (346.9, 171.3)
- added ?: , components:diode-silk, B.Cu at (303.8, 169.9)
- added ?: , components:diode-silk, B.Cu at (304.0, 161.7)
- added ?: , components:diode-silk, B.Cu at (273.7, 161.0)
- added ?: , components:diode-silk, B.Cu at (267.5, 167.3)
- added ?: , components:diode-silk, B.Cu at (254.2, 161.0)
- added ?: , components:diode-silk, B.Cu at (234.8, 160.7)
- added ?: , components:diode-silk, B.Cu at (240.6, 168.7)
- added ?: , components:diode-silk, B.Cu at (79.5, 183.4)
- added ?: , components:diode-silk, B.Cu at (221.6, 169.1)
- added ?: , components:diode-silk, B.Cu at (215.9, 160.6)
- added ?: , components:diode-silk, B.Cu at (197.2, 160.3)
- added ?: , components:diode-silk, B.Cu at (202.4, 169.0)
- added ?: , components:diode-silk, B.Cu at (183.3, 168.7)
- added ?: , components:diode-silk, B.Cu at (177.8, 160.3)
- added ?: , components:diode-silk, B.Cu at (158.9, 160.3)
- added ?: , components:diode-silk, B.Cu at (164.2, 168.4)
- added ?: , components:diode-silk, B.Cu at (145.2, 168.7)
- added ?: , components:diode-silk, B.Cu at (140.0, 160.1)
- added ?: , components:diode-silk, B.Cu at (103.4, 183.3)
- added ?: , components:diode-silk, B.Cu at (120.9, 160.1)
- added ?: , components:diode-silk, B.Cu at (126.2, 168.3)
- added ?: , components:diode-silk, B.Cu at (106.0, 167.1)
- added ?: , components:diode-silk, B.Cu at (102.0, 159.8)
- added ?: , components:diode-silk, B.Cu at (82.9, 160.0)
- added ?: , components:diode-silk, B.Cu at (88.0, 167.8)
- added ?: , components:diode-silk, B.Cu at (63.1, 165.6)
- added ?: , components:diode-silk, B.Cu at (56.6, 160.1)
- added ?: , components:diode-silk, B.Cu at (372.2, 130.4)
- added ?: , components:diode-silk, B.Cu at (355.0, 129.7)
- added ?: , components:diode-silk, B.Cu at (173.0, 183.5)
- added ?: , components:diode-silk, B.Cu at (341.9, 129.9)
- added ?: , components:diode-silk, B.Cu at (314.5, 131.1)
- added ?: , components:diode-silk, B.Cu at (283.4, 131.4)
- added ?: , components:diode-silk, B.Cu at (264.4, 131.2)
- added ?: , components:diode-silk, B.Cu at (245.0, 130.9)
- added ?: , components:diode-silk, B.Cu at (226.2, 130.4)
- added ?: , components:diode-silk, B.Cu at (207.1, 130.1)
- added ?: , components:diode-silk, B.Cu at (188.1, 130.9)
- added ?: , components:diode-silk, B.Cu at (169.0, 130.6)
- added ?: , components:diode-silk, B.Cu at (150.0, 130.1)
- added ?: , components:diode-silk, B.Cu at (244.9, 184.7)
- added ?: , components:diode-silk, B.Cu at (130.9, 130.5)
- added ?: , components:diode-silk, B.Cu at (111.9, 130.0)
- added ?: , components:diode-silk, B.Cu at (54.3, 124.1)
- added ?: , components:diode-silk, B.Cu at (56.5, 131.9)
- added ?: , components:diode-silk, B.Cu at (92.5, 129.3)
- added ?: , components:diode-silk, B.Cu at (73.5, 129.9)
- added ?: , components:diode-silk, B.Cu at (68.2, 124.2)
- added ?: , components:diode-silk, B.Cu at (87.2, 124.3)
- added ?: , components:diode-silk, B.Cu at (106.7, 124.4)
- added ?: , components:diode-silk, B.Cu at (125.2, 123.5)
- added ?: , components:diode-silk, B.Cu at (268.4, 183.3)
- added ?: , components:diode-silk, B.Cu at (144.5, 123.4)
- added ?: , components:diode-silk, B.Cu at (163.6, 123.1)
- added ?: , components:diode-silk, B.Cu at (182.5, 122.8)
- added ?: , components:diode-silk, B.Cu at (201.7, 122.6)
- added ?: , components:diode-silk, B.Cu at (220.8, 122.5)
- added ?: , components:diode-silk, B.Cu at (239.5, 122.6)
- added ?: , components:diode-silk, B.Cu at (259.1, 122.6)
- added ?: , components:diode-silk, B.Cu at (278.3, 122.4)
- added ?: , components:diode-silk, B.Cu at (306.6, 122.7)
- added ?: , components:diode-silk, B.Cu at (340.0, 122.7)
- added ?: , components:diode-silk, B.Cu at (292.6, 187.8)
- added ?: , components:diode-silk, B.Cu at (359.0, 122.4)
- added ?: , components:diode-silk, B.Cu at (370.3, 122.3)
- added ?: , components:diode-silk, B.Cu at (373.6, 83.7)
- added ?: , components:diode-silk, B.Cu at (354.8, 83.2)
- added ?: , components:diode-silk, B.Cu at (341.5, 80.6)
- added ?: , components:diode-silk, B.Cu at (310.5, 82.1)
- added ?: , components:diode-silk, B.Cu at (296.9, 95.9)
- added ?: , components:diode-silk, B.Cu at (282.8, 96.0)
- added ?: , components:diode-silk, B.Cu at (263.8, 96.0)
- added ?: , components:diode-silk, B.Cu at (235.3, 96.0)
- added ?: , components:diode-silk, B.Cu at (317.1, 187.5)
- added ?: , components:diode-silk, B.Cu at (216.2, 96.0)
- added ?: , components:diode-silk, B.Cu at (197.1, 96.0)
- added ?: , components:diode-silk, B.Cu at (178.2, 96.1)
- added ?: , components:diode-silk, B.Cu at (149.6, 96.1)
- added ?: , components:diode-silk, B.Cu at (130.7, 96.0)
- added ?: , components:diode-silk, B.Cu at (111.4, 96.0)
- added ?: , components:diode-silk, B.Cu at (92.2, 95.9)
- added ?: , components:diode-silk, B.Cu at (54.4, 95.8)
- added ?: , components:diode-silk, B.Cu at (335.7, 188.2)

Commit message: refined silkscreens
Parts:
- removed ? (x87): , components:diode-silk
- added G***: LOGO, components:Apex-silk, F.Cu at (325.3, 172.6)
- moved R13 2.86 mm to (74.5, 74.4)
- moved C19 1.91 mm to (56.6, 76.0)
Routing:
- net Net-(C19-Pad2): track 7.06 -> 8.25 mm
Other:
- board text added: "."
- board text added: "D+"
- board text added: "D-"
- board text added: "ENCODER"
- board text added: "GND"
- board text added: "Rev. 1 Rev. Date 7.20.20 Designed by /jastein91 https://github.com/jstein91/Apex"
- board text added: "SCL"
- board text added: "SDA"
- board text added: "VCC"

Commit message: Fill zones
Removed large fill zone and created one small one for XTAL area and larger one for whole board
Parts:
- moved C2 1.49 mm to (361.8, 162.0)
- moved C1 0.72 mm to (355.0, 161.9)
Routing:
- net GND: track 97.0 -> 182.3 mm, vias 10 -> 16
- net Net-(C1-Pad1): track 7.55 -> 6.82 mm
